File: TesterSchema/Część fizyczna/v1.1/Tester ogniw v1.1 - Moduł mocy.kicad_pcb (KiCad board)
At the start: 2 copper layers, 182 x 75 mm, 42 parts, among them J1 J2, K1 K10, K3 Zasilanie, K4 Badany AKU, T1 IRFP9140, T2 IRFP054N, T3 BC547, T4 BC547, T5 T_PNP, T6 BC547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

Commit message: Poprawienie schematu Sterownika w związku z migracją na KiCAD2015 Poprawienie schematu Modułu Mocy w związku z migracją na KiCAD2015 i dodaniem clamp'a na wyjściu AKU
Parts:
- R10, R11, R13, R14, R5, R7, R8, R9: footprint resistor-0207/7 -> 7:
- R12, R24, R6: footprint resistor-0207/10 -> 10:

Commit message: naprawa pliku PCB modułu mocy
Parts:
- R10, R11, R13, R14, R5, R7, R8, R9: footprint 7: -> resistor-0207/7
- R12, R24, R6: footprint 10: -> resistor-0207/10
Changed lines of the file:
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@@
       (net 15 N-0000018))
   )
-  (module 7: (layer B.Cu)
+  (module resistor-0207/7 (layer B.Cu)
     (at 225.25 102.5 90)
     (descr RESISTOR)
@@
       (net 10 N-0000010))
   )
-  (module 10: (layer B.Cu)
+  (module resistor-0207/10 (layer B.Cu)
     (at 288.75 86.25 180)
     (descr RESISTOR)
@@
     )
   )
-  (module 7: (layer F.Cu)
+  (module resistor-0207/7 (layer F.Cu)
     (at 178.75 75.25 180)
     (descr RESISTOR)
@@
       (net 30 N-000006))
   )
-  (module 7: (layer F.Cu)
+  (module resistor-0207/7 (layer F.Cu)
     (at 340.5 76.25 180)
     (descr RESISTOR)
@@
       (net 31 N-000007))
   )
-  (module 7: (layer B.Cu)
+  (module resistor-0207/7 (layer B.Cu)
     (at 218.25 115.25 180)
     (descr RESISTOR)
@@
       (net 11 N-0000013))
   )
-  (module 7: (layer B.Cu)
+  (module resistor-0207/7 (layer B.Cu)
     (at 218.25 107.75)
     (descr RESISTOR)
@@
       (net 10 N-0000010))
   )
-  (module 7: (layer B.Cu)
+  (module resistor-0207/7 (layer B.Cu)
     (at 218.25 112.75 180)
     (descr RESISTOR)
@@
       (net 13 N-0000016))
   )
-  (module 7: (layer B.Cu)
+  (module resistor-0207/7 (layer B.Cu)
     (at 218.25 110.25 180)
     (descr RESISTOR)
@@
       (net 33 N-000009))
   )
-  (module 7: (layer B.Cu)
+  (module resistor-0207/7 (layer B.Cu)
     (at 288.75 83.5)
     (descr RESISTOR)
@@
       (net 32 N-000008))
   )
-  (module 10: (layer F.Cu)
+  (module resistor-0207/10 (layer F.Cu)
     (at 341.75 73.25 180)
     (descr RESISTOR)
@@
       (net 1 /+18V))
   )
-  (module 10: (layer F.Cu)
+  (module resistor-0207/10 (layer F.Cu)
     (at 180 72.5 180)
     (descr RESISTOR)

Commit message: Naprawa repo
Parts:
- R10, R11, R13, R14, R5, R7, R8, R9: footprint resistor-0207/7 -> resistor-0207_7
- R12, R24, R6: footprint resistor-0207/10 -> resistor-0207_10
Changed lines of the file:
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@@
       (net 15 N-0000018))
   )
-  (module resistor-0207/7 (layer B.Cu)
+  (module resistor-0207_7 (layer B.Cu)
     (at 225.25 102.5 90)
     (descr RESISTOR)
@@
       (net 10 N-0000010))
   )
-  (module resistor-0207/10 (layer B.Cu)
+  (module resistor-0207_10 (layer B.Cu)
     (at 288.75 86.25 180)
     (descr RESISTOR)
@@
     )
   )
-  (module resistor-0207/7 (layer F.Cu)
+  (module resistor-0207_7 (layer F.Cu)
     (at 178.75 75.25 180)
     (descr RESISTOR)
@@
       (net 30 N-000006))
   )
-  (module resistor-0207/7 (layer F.Cu)
+  (module resistor-0207_7 (layer F.Cu)
     (at 340.5 76.25 180)
     (descr RESISTOR)
@@
       (net 31 N-000007))
   )
-  (module resistor-0207/7 (layer B.Cu)
+  (module resistor-0207_7 (layer B.Cu)
     (at 218.25 115.25 180)
     (descr RESISTOR)
@@
       (net 11 N-0000013))
   )
-  (module resistor-0207/7 (layer B.Cu)
+  (module resistor-0207_7 (layer B.Cu)
     (at 218.25 107.75)
     (descr RESISTOR)
@@
       (net 10 N-0000010))
   )
-  (module resistor-0207/7 (layer B.Cu)
+  (module resistor-0207_7 (layer B.Cu)
     (at 218.25 112.75 180)
     (descr RESISTOR)
@@
       (net 13 N-0000016))
   )
-  (module resistor-0207/7 (layer B.Cu)
+  (module resistor-0207_7 (layer B.Cu)
     (at 218.25 110.25 180)
     (descr RESISTOR)
@@
       (net 33 N-000009))
   )
-  (module resistor-0207/7 (layer B.Cu)
+  (module resistor-0207_7 (layer B.Cu)
     (at 288.75 83.5)
     (descr RESISTOR)
@@
       (net 32 N-000008))
   )
-  (module resistor-0207/10 (layer F.Cu)
+  (module resistor-0207_10 (layer F.Cu)
     (at 341.75 73.25 180)
     (descr RESISTOR)
@@
       (net 1 /+18V))
   )
-  (module resistor-0207/10 (layer F.Cu)
+  (module resistor-0207_10 (layer F.Cu)
     (at 180 72.5 180)
     (descr RESISTOR)
