File: TesterSchema/Część fizyczna/v1.1/_autosave-Tester ogniw v1.1 - Sterownik.kicad_pcb (KiCad board)
At the start: 2 copper layers, 75 x 100 mm, 82 parts, among them K1 D-SUB-DE-9, K2 JTAG-ATMEL, K3 K20, K4 K10, P2 500R, P3 1k, P4 100k, T1 BC547, T2 BC547, U1 TL082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

Commit message: Poprawienie schematu Sterownika w związku z migracją na KiCAD2015 Poprawienie schematu Modułu Mocy w związku z migracją na KiCAD2015 i dodaniem clamp'a na wyjściu AKU
Parts:
- R1: footprint resistor-0204/5 -> 5:
- R22: footprint resistor-0207/7 -> 7:
- R28: footprint resistor-0207/2V -> 2V:
Routing:
- net /TCK: track 9.22 -> 0.00 mm
- net N-0000050: track 8.53 -> 12.2 mm
- net /DSG: track 55.3 -> 51.6 mm

Commit message: Naprawa repo
Parts:
- R22: footprint 7: -> resistor-0207_7
- R28: footprint 2V: -> resistor-0207_2V
Changed lines of the file:
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@@
       (net 43 GND))
   )
-  (module 2V: (layer Gorna)
+  (module resistor-0207_2V (layer Gorna)
     (at 144.5 96.2 270)
     (descr RESISTOR)
@@
     )
   )
-  (module 7: (layer Gorna)
+  (module resistor-0207_7 (layer Gorna)
     (at 174.2 67 90)
     (descr RESISTOR)
