File: TesterSchema/Część fizyczna/v1.0/Tester ogniw v1.0.kicad_pcb (KiCad board)
At the start: 2 copper layers, 104 parts, among them K1 D-SUB-DE-9, K2 JTAG-ATMEL, K3 Zasilanie, K4 Badany AKU, P1 P, P2 500R, P3 P, P4 100k, SW1 SW, SW2 SW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

Commit message: Naprawa repo
Parts:
- R22: footprint resistor-0207/7 -> resistor-0207_7
- R28: footprint resistor-0207/2V -> resistor-0207_2V
Changed lines of the file:
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@@
     )
   )
-  (module resistor-0207/2V (layer Gorna)
+  (module resistor-0207_2V (layer Gorna)
     (at 134.3 155.6 270)
     (descr RESISTOR)
@@
     )
   )
-  (module resistor-0207/7 (layer Gorna)
+  (module resistor-0207_7 (layer Gorna)
     (at 160.7 128.3 90)
     (descr RESISTOR)
