File: TesterSchema/atxmega32a4_adapter/atxmega_adapter.kicad_pcb (KiCad board)
At the start: 2 copper layers, 55 x 20 mm, 29 parts, among them IC1 ATXMEGA32A4-M, P1 DIL40, Q1 BC817-40, Q2 BC817-40, Q3 BC817-40, U1 APE8865N-33-HF-3

Commit message: Zmiana nazwy stabilizatore/ poprawki w adapeerze
Routing:
- net GND: track 126.1 -> 130.2 mm
- net /SW4: track 39.2 -> 40.8 mm
- net +3.3V: track 135.7 -> 137.1 mm
